Commit message: -

File: Master node/moveo6_support/moveo6/moveo6.urdf (robot description, URDF)
Before this commit: robot moveo6, 8 links, 7 joints
Links:
- added link moveo6_base
Joints:
- added joint moveo6base_link-base: type fixed, parent base_link, child moveo6_base, origin xyz= 0 0 0 rpy=0 0 0 

Commit message: -

File: Master node/moveo6_support/moveo6/moveo6.urdf (robot description, URDF)
Before this commit: robot moveo6, 9 links, 8 joints
Links:
- removed link moveo6_base
- link base_link: mass 10.579237 -> None
Joints:
- removed joint moveo6base_link-base

Commit message: -

File: Master node/moveo6_support/moveo6/moveo6.urdf (robot description, URDF)
Before this commit: robot moveo6, 8 links, 7 joints
Links:
- removed link moveo_1_1
- removed link moveo_2_1
- removed link moveo_3_1
- removed link moveo_4_1
- removed link moveo_5_1
- removed link moveo_6_1
- removed link moveo_7_1
- added link base
- added link link_1, mass 2.573085; collision mesh filename=package://moveo6_support/moveo6/bin_stl/moveo_1_1_m-binary.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; visual mesh filename=package://moveo6_support/moveo6/bin_stl/moveo_1_1_m-binary.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
- added link link_2, mass 9.981201; collision mesh filename=package://moveo6_support/moveo6/bin_stl/moveo_2_1_m-binary.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; visual mesh filename=package://moveo6_support/moveo6/bin_stl/moveo_2_1_m-binary.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
- added link link_3, mass 14.019629; collision mesh filename=package://moveo6_support/moveo6/bin_stl/moveo_3_1_m-binary.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; visual mesh filename=package://moveo6_support/moveo6/bin_stl/moveo_3_1_m-binary.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
- added link link_4, mass 5.138963; collision mesh filename=package://moveo6_support/moveo6/bin_stl/moveo_4_1_m-binary.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; visual mesh filename=package://moveo6_support/moveo6/bin_stl/moveo_4_1_m-binary.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
- added link link_5, mass 2.051396; collision mesh filename=package://moveo6_support/moveo6/bin_stl/moveo_5_1_m-binary.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; visual mesh filename=package://moveo6_support/moveo6/bin_stl/moveo_5_1_m-binary.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
- added link link_6, mass 1.487313; collision mesh filename=package://moveo6_support/moveo6/bin_stl/moveo_6_1_m-binary.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; visual mesh filename=package://moveo6_support/moveo6/bin_stl/moveo_6_1_m-binary.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
- added link link_7, mass 0.332399; collision mesh filename=package://moveo6_support/moveo6/bin_stl/moveo_7_1_m-binary.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; visual mesh filename=package://moveo6_support/moveo6/bin_stl/moveo_7_1_m-binary.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
Joints:
- removed joint Rev1
- removed joint Rev3
- removed joint Rev5
- removed joint Rev6
- removed joint Rev7
- removed joint Rigid13
- removed joint rev4
- added joint base_link-base: type fixed, parent $base_link, child base, origin xyz=0 0 0 rpy=0 0 0
- added joint joint_1: type revolute, parent base_link, child joint_1, origin xyz=0.0 0.0 0.065 rpy=0 0 0, axis -0.0 0.0 0.01, limit lower=-3.141593 upper=3.141593 effort=100 velocity=100
- added joint joint_2: type revolute, parent link_2, child link_3, origin xyz=-0.06 0.0 0.14 rpy=0 0 0, axis -0.01 0.0 -0.0, limit lower=-1.919862 upper=1.832596 effort=100 velocity=100
- added joint joint_3: type revolute, parent link_3, child link_4, origin xyz=0.0885 0.006028 0.221042 rpy=0 0 0, axis 0.01 -0.0 0.0, limit lower=-2.443461 upper=2.181662 effort=100 velocity=100
- added joint joint_4: type revolute, parent link_4, child link_5, origin xyz=-0.03675 0.024328 0.125157 rpy=0 0 0, axis 0.0 0.001908 0.009816, limit lower=0.0 upper=6.283185 effort=100 velocity=100
- added joint joint_5: type revolute, parent link_5, child link_6, origin xyz=-0.024994 0.017585 0.09336 rpy=0 0 0, axis -0.009998 -0.000217 4.2e-05, limit lower=-1.832596 upper=2.007129 effort=100 velocity=100
- added joint joint_6: type revolute, parent link_6, child link_7, origin xyz=0.024081 0.007333 0.055483 rpy=0 0 0, axis 1.5e-05 0.001217 0.009926, limit lower=-5.148721 upper=0.959931 effort=100 velocity=100
- added joint rigid_joint_1-2: type fixed, parent link_1, child link_2, origin xyz=0.0 0.0 0.0255 rpy=0 0 0

Commit message: Fixed the URDF and the model finally works

File: Master node/moveo6_support/moveo6/moveo6.urdf (robot description, URDF)
Before this commit: robot moveo6, 9 links, 8 joints
Links:
- link base_link: mass 10.579237 -> None
Joints:
- joint base_link-base: parent $base_link -> base_link
- joint joint_1: child joint_1 -> link_1
